File: hardware/prototype/hmi_board/hmi_keypad.kicad_sch (KiCad schematic)
At the start: 33 parts, among them SW401 SW_A1, SW402 SW_A2, SW403 SW_A3, SW404 SW_A4, SW411 SW_B1, SW412 SW_B2, SW413 SW_B3, SW414 SW_B4, SW421 SW_C1, SW422 SW_C2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

Commit message: Added column jumpers
Parts:
- added JP401, JP402, JP403, JP404: SolderJumper_3_Bridged12, symbol Jumper:SolderJumper_3_Bridged12
Connections:
- net COL_1: now also JP401.3 (B); no longer R401.2, R411.2, R421.2, R431.2
- net COL_2: now also JP402.3 (B); no longer R402.2, R412.2, R422.2, R432.2
- net COL_3: now also JP403.3 (B); no longer R403.2, R413.2, R423.2, R433.2
- net COL_4: now also JP404.3 (B); no longer R404.2, R408.2, R412.2, R434.2
- net GND: now also JP401.2 (C), JP402.2 (C), JP403.2 (C), JP404.2 (C)
- new net COL_1L: JP401.1 (A), R401.2, R411.2, R421.2, R431.2
- new net COL_2L: JP402.1 (A), R402.2, R412.2, R422.2, R432.2
- new net COL_3L: JP403.1 (A), R403.2, R413.2, R423.2, R433.2
- new net COL_4L: JP404.1 (A), R404.2, R408.2, R412.2, R434.2
Other:
- note added: "Key matrix is intended to be possible to wire using either: - Scanning Row/Column matrix - Resistor divider with columns tied to ground and PU resistor on Row Jumpers are defaulted to the resistor divider approach."
- note removed: "Key matrix is intended to be possible to wire using either: - Scanning Row/Column matrix - Resistor divider with columns tied to ground and PU resistor on Row"

Commit message: Add display board
Parts:
- JP401: value SolderJumper_3_Bridged12 -> Col 1 Jumper; footprint (none) -> Jumper:SolderJumper-3_P1.3mm_Bridged12_RoundedPad1.0x1.5mm_NumberLabels
- JP402: value SolderJumper_3_Bridged12 -> Col 2 Jumper; footprint (none) -> Jumper:SolderJumper-3_P1.3mm_Bridged12_RoundedPad1.0x1.5mm_NumberLabels
- JP403: value SolderJumper_3_Bridged12 -> Col 3 Jumper; footprint (none) -> Jumper:SolderJumper-3_P1.3mm_Bridged12_RoundedPad1.0x1.5mm_NumberLabels
- JP404: value SolderJumper_3_Bridged12 -> Col 4 Jumper; footprint (none) -> Jumper:SolderJumper-3_P1.3mm_Bridged12_RoundedPad1.0x1.5mm_NumberLabels
Other:
- moved on the sheet: JP402, JP403, JP404
Changed lines of the file:
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@@
 	(wire
 		(pts
-			(xy 229.87 60.96) (xy 234.95 60.96)
+			(xy 228.6 54.61) (xy 233.68 54.61)
 		)
 		(stroke
@@
 	(wire
 		(pts
-			(xy 245.11 106.68) (xy 248.92 106.68)
+			(xy 243.84 97.79) (xy 247.65 97.79)
 		)
 		(stroke
@@
 	(wire
 		(pts
-			(xy 243.84 82.55) (xy 247.65 82.55)
+			(xy 243.84 76.2) (xy 247.65 76.2)
 		)
 		(stroke
@@
 	(wire
 		(pts
-			(xy 240.03 64.77) (xy 240.03 67.31)
+			(xy 238.76 58.42) (xy 238.76 60.96)
 		)
 		(stroke
@@
 	(wire
 		(pts
-			(xy 238.76 86.36) (xy 238.76 88.9)
+			(xy 238.76 80.01) (xy 238.76 82.55)
 		)
 		(stroke
@@
 	(wire
 		(pts
-			(xy 245.11 60.96) (xy 248.92 60.96)
+			(xy 243.84 54.61) (xy 247.65 54.61)
 		)
 		(stroke
@@
 	(wire
 		(pts
-			(xy 240.03 110.49) (xy 240.03 114.3)
+			(xy 238.76 101.6) (xy 238.76 105.41)
 		)
 		(stroke
@@
 	(wire
 		(pts
-			(xy 229.87 106.68) (xy 234.95 106.68)
+			(xy 228.6 97.79) (xy 233.68 97.79)
 		)
 		(stroke
@@
 	(wire
 		(pts
-			(xy 228.6 82.55) (xy 233.68 82.55)
+			(xy 228.6 76.2) (xy 233.68 76.2)
 		)
 		(stroke
@@
 	)
 	(label "COL_3L"
-		(at 228.6 82.55 180)
+		(at 228.6 76.2 180)
 		(effects
 			(font
@@
 	)
 	(label "COL_4L"
-		(at 229.87 106.68 180)
+		(at 228.6 97.79 180)
 		(effects
 			(font
@@
 	)
 	(label "COL_2L"
-		(at 229.87 60.96 180)
+		(at 228.6 54.61 180)
 		(effects
 			(font
@@
 	(hierarchical_label "COL_2"
 		(shape input)
-		(at 248.92 60.96 0)
+		(at 247.65 54.61 0)
 		(effects
 			(font
@@
 	(hierarchical_label "COL_3"
 		(shape input)
-		(at 247.65 82.55 0)
+		(at 247.65 76.2 0)
 		(effects
 			(font
@@
 	(hierarchical_label "COL_4"
 		(shape input)
-		(at 248.92 106.68 0)
+		(at 247.65 97.79 0)
 		(effects
 			(font
@@
 	(symbol
 		(lib_id "Jumper:SolderJumper_3_Bridged12")
-		(at 238.76 82.55 0)
+		(at 238.76 76.2 0)
 		(unit 1)
 		(exclude_from_sim no)
@@
 		(fields_autoplaced yes)
 		(property "Reference" "JP403"
-			(at 238.76 76.2 0)
+			(at 238.76 69.85 0)
 			(effects
 				(font
@@
 			)
 		)
-		(property "Value" "SolderJumper_3_Bridged12"
-			(at 238.76 78.74 0)
+		(property "Value" "Col 3 Jumper"
+			(at 238.76 72.39 0)
 			(effects
 				(font
@@
 			)
 		)
-		(property "Footprint" ""
-			(at 238.76 82.55 0)
+		(property "Footprint" "Jumper:SolderJumper-3_P1.3mm_Bridged12_RoundedPad1.0x1.5mm_NumberLabels"
+			(at 238.76 76.2 0)
 			(effects
 				(font
@@
 		)
 		(property "Datasheet" "~"
-			(at 238.76 82.55 0)
+			(at 238.76 76.2 0)
 			(effects
 				(font
@@
 		)
 		(property "Description" "3-pole Solder Jumper, pins 1+2 closed/bridged"
-			(at 238.76 82.55 0)
+			(at 238.76 76.2 0)
 			(effects
 				(font
@@
 	(symbol
 		(lib_id "Jumper:SolderJumper_3_Bridged12")
-		(at 240.03 106.68 0)
+		(at 238.76 97.79 0)
 		(unit 1)
 		(exclude_from_sim no)
@@
 		(fields_autoplaced yes)
 		(property "Reference" "JP404"
-			(at 240.03 100.33 0)
+			(at 238.76 91.44 0)
 			(effects
 				(font
@@
 			)
 		)
-		(property "Value" "SolderJumper_3_Bridged12"
-			(at 240.03 102.87 0)
+		(property "Value" "Col 4 Jumper"
+			(at 238.76 93.98 0)
 			(effects
 				(font
@@
 			)
 		)
-		(property "Footprint" ""
-			(at 240.03 106.68 0)
+		(property "Footprint" "Jumper:SolderJumper-3_P1.3mm_Bridged12_RoundedPad1.0x1.5mm_NumberLabels"
+			(at 238.76 97.79 0)
 			(effects
 				(font
@@
 		)
 		(property "Datasheet" "~"
-			(at 240.03 106.68 0)
+			(at 238.76 97.79 0)
 			(effects
 				(font
@@
 		)
 		(property "Description" "3-pole Solder Jumper, pins 1+2 closed/bridged"
-			(at 240.03 106.68 0)
+			(at 238.76 97.79 0)
 			(effects
 				(font
@@
 	(symbol
 		(lib_id "power:GND")
-		(at 238.76 88.9 0)
+		(at 238.76 82.55 0)
 		(unit 1)
 		(exclude_from_sim no)
@@
 		(fields_autoplaced yes)
 		(property "Reference" "#PWR0404"
-			(at 238.76 95.25 0)
+			(at 238.76 88.9 0)
 			(effects
 				(font
@@
 		)
 		(property "Value" "GND"
-			(at 238.76 93.98 0)
+			(at 238.76 87.63 0)
 			(effects
 				(font
@@
 		)
 		(property "Footprint" ""
-			(at 238.76 88.9 0)
+			(at 238.76 82.55 0)
 			(effects
 				(font
@@
 		)
 		(property "Datasheet" ""
-			(at 238.76 88.9 0)
+			(at 238.76 82.55 0)
 			(effects
 				(font
@@
 		)
 		(property "Description" "Power symbol creates a global label with name \"GND\" , ground"
-			(at 238.76 88.9 0)
+			(at 238.76 82.55 0)
 			(effects
 				(font
@@
 	(symbol
 		(lib_id "Jumper:SolderJumper_3_Bridged12")
-		(at 240.03 60.96 0)
+		(at 238.76 54.61 0)
 		(unit 1)
 		(exclude_from_sim no)
@@
 		(fields_autoplaced yes)
 		(property "Reference" "JP402"
-			(at 240.03 54.61 0)
+			(at 238.76 48.26 0)
 			(effects
 				(font
@@
 			)
 		)
-		(property "Value" "SolderJumper_3_Bridged12"
-			(at 240.03 57.15 0)
+		(property "Value" "Col 2 Jumper"
+			(at 238.76 50.8 0)
 			(effects
 				(font
@@
 			)
 		)
-		(property "Footprint" ""
-			(at 240.03 60.96 0)
+		(property "Footprint" "Jumper:SolderJumper-3_P1.3mm_Bridged12_RoundedPad1.0x1.5mm_NumberLabels"
+			(at 238.76 54.61 0)
 			(effects
 				(font
@@
 		)
 		(property "Datasheet" "~"
-			(at 240.03 60.96 0)
+			(at 238.76 54.61 0)
 			(effects
 				(font
@@
 		)
 		(property "Description" "3-pole Solder Jumper, pins 1+2 closed/bridged"
-			(at 240.03 60.96 0)
+			(at 238.76 54.61 0)
 			(effects
 				(font
@@
 			)
 		)
-		(property "Value" "SolderJumper_3_Bridged12"
+		(property "Value" "Col 1 Jumper"
 			(at 238.76 29.21 0)
 			(effects
@@
 			)
 		)
-		(property "Footprint" ""
+		(property "Footprint" "Jumper:SolderJumper-3_P1.3mm_Bridged12_RoundedPad1.0x1.5mm_NumberLabels"
 			(at 238.76 33.02 0)
 			(effects
@@
 	(symbol
 		(lib_id "power:GND")
-		(at 240.03 114.3 0)
+		(at 238.76 105.41 0)
 		(unit 1)
 		(exclude_from_sim no)
@@
 		(fields_autoplaced yes)
 		(property "Reference" "#PWR0405"
-			(at 240.03 120.65 0)
+			(at 238.76 111.76 0)
 			(effects
 				(font
@@
 		)
 		(property "Value" "GND"
-			(at 240.03 119.38 0)
+			(at 238.76 110.49 0)
 			(effects
 				(font
@@
 		)
 		(property "Footprint" ""
-			(at 240.03 114.3 0)
+			(at 238.76 105.41 0)
 			(effects
 				(font
@@
 		)
 		(property "Datasheet" ""
-			(at 240.03 114.3 0)
+			(at 238.76 105.41 0)
 			(effects
 				(font
@@
 		)
 		(property "Description" "Power symbol creates a global label with name \"GND\" , ground"
-			(at 240.03 114.3 0)
+			(at 238.76 105.41 0)
 			(effects
 				(font
@@
 	(symbol
 		(lib_id "power:GND")
-		(at 240.03 67.31 0)
+		(at 238.76 60.96 0)
 		(unit 1)
 		(exclude_from_sim no)
@@
 		(fields_autoplaced yes)
 		(property "Reference" "#PWR0403"
-			(at 240.03 73.66 0)
+			(at 238.76 67.31 0)
 			(effects
 				(font
@@
 		)
 		(property "Value" "GND"
-			(at 240.03 72.39 0)
+			(at 238.76 66.04 0)
 			(effects
 				(font
@@
 		)
 		(property "Footprint" ""
-			(at 240.03 67.31 0)
+			(at 238.76 60.96 0)
 			(effects
 				(font
@@
 		)
 		(property "Datasheet" ""
-			(at 240.03 67.31 0)
+			(at 238.76 60.96 0)
 			(effects
 				(font
@@
 		)
 		(property "Description" "Power symbol creates a global label with name \"GND\" , ground"
-			(at 240.03 67.31 0)
+			(at 238.76 60.96 0)
 			(effects
 				(font
