File: hardware/prototype/hmi_board/hmi_microcontroller.kicad_sch (KiCad schematic)
At the start: 1 part, among them U101 ATSAMD10D13A-M

Commit message: Add display board
Connections:
- net COL_1: now also U101.11 (PA14)
- net COL_2: now also U101.12 (PA15)
- net COL_3: now also U101.13 (PA16)
- net COL_4: now also U101.14 (PA17)
- net INT: now also U101.21 (PA24)
- net NAV_A: now also U101.6 (PA07)
- net NAV_B: now also U101.9 (PA10)
- net NAV_DIR: now also U101.5 (PA06)
- net NAV_SW: now also U101.10 (PA11)
- net POW_SW: now also U101.17 (PA27)
- net ROW_A: now also U101.1 (PA02)
- net ROW_B: now also U101.2 (PA03)
- net ROW_C: now also U101.3 (PA04)
- net ROW_D: now also U101.4 (PA05)
- net SCL: now also U101.16 (PA23)
- net SDA: now also U101.15 (PA22)
- net WAKE: now also U101.22 (PA25)
Other:
- note added: "Clocks: - Internal 48MHz clock"
- note added: "Pin Assignment Considerations: - Rows must be analog capable for resistor divider keyboard - NAV_DIR must be analog capable for resistor divider approach - NAV_A or NAV_B must be interrupt capable to pick up quadrature direction - Power switch must be capable of waking up the system from STANDBY"
