File: hardware/prototype/hmi_board/hmi_board.kicad_sch (KiCad schematic)
At the start: 2 parts, among them J101 PGM, J102 Host

Commit message: Combined board started
Parts:
- removed J102: Host, symbol Connector_Generic:Conn_01x06
- added J101: HOST, symbol Connector_Generic:Conn_01x07
- renumbered J101 to J102
Connections:
- net +3.3V: now also J101.2 (Pin_2)
- net GND: now also J101.1 (Pin_1)
- net Microcontroller/INT: now also J101.6 (Pin_6)
- net Microcontroller/SCL: now also J101.4 (Pin_4)
- net Microcontroller/SDA: now also J101.5 (Pin_5)
- net Microcontroller/WAKE: now also J101.7 (Pin_7)
- new net +5V: J101.3 (Pin_3)
Other:
- added sheet VFO (hmi_vfo.kicad_sch)
- sheet Keypad ports: added RGB_DATA; removed COL_1, COL_2, COL_3, COL_4
- sheet Microcontroller ports: added RGB_DATA, VFO_A, VFO_ADJ_A, VFO_ADJ_B, VFO_B, VFO_SW; removed COL_1, COL_2, COL_3, COL_4
- note added: "+5V is unregulated battery voltage Can range from battery cutoff voltage to +4.5V"
