File: hardware/prototype/display_board/display_board.kicad_sch (KiCad schematic)
At the start: 0 parts

Commit message: Combined board started
Parts:
- added J101: HMI, symbol Connector_Generic:Conn_01x07
Connections:
- new net +3.3V: J101.2 (Pin_2)
- new net +5V: J101.3 (Pin_3)
- new net GND: J101.1 (Pin_1)
- new net HMI_I2C_SCL: J101.4 (Pin_4)
- new net HMI_I2C_SDA: J101.5 (Pin_5)
- new net Microcontroller/HMI_INT: J101.6 (Pin_6)
- new net Microcontroller/HMI_WAKE: J101.7 (Pin_7)
- no-connect marks 0 -> 1
Other:
- added sheet Audio (mpu_audio.kicad_sch)
- added sheet Battery (display_battery.kicad_sch)
- added sheet Power Regulation (mcu_power.kicad_sch)
- sheet Display Connectors ports: added DISP_BL, DISP_CS, DISP_DC, DISP_RST, DISP_SCL, DISP_SDA, DISP_TS_INT, DISP_TS_RST, DISP_TS_SCL, DISP_TS_SDA; removed none
- sheet Microcontroller ports: added DISP_BL, DISP_CS, DISP_DC, DISP_RST, DISP_SCL, DISP_SDA, DISP_TS_INT, DISP_TS_RST, HMI_INT, HMI_WAKE, I2C_SCK, I2C_SDA, I2S_ADCIN, I2S_ADCOUT, I2S_BCLK, I2S_FS, I2S_MCLK, PWR_CHRG, PWR_EXT, V_usb; removed none
- note added: "I2C Bus Addresses NAU8822 Codec: 0x19 Touch Controller: HMI Board: Undecided, can be any"
