File: hardware/prototype/minstro_combined_board/hmi_keypad.kicad_sch (KiCad schematic)
At the start: 49 parts, among them SW901 SW_A1, SW902 SW_A2, SW903 SW_A3, SW904 SW_A4, SW905 SW_B1, SW906 SW_B2, SW907 SW_B3, SW908 SW_B4, SW909 SW_C1, SW910 SW_C2, SW911 SW_C3, SW912 SW_C4, SW913 SW_D1, SW914 SW_D2, SW915 SW_D3, SW916 SW_D4, SW917 POWER

Commit message: Layout WIP
Parts:
- removed D901, D902, D903, D904, D905, D906, D907, D908, D909, D910, D911, D912, D913, D914, D915, D916: ~, BVH_LED:SK6812Mini-E_Front, symbol BVH_LED:WS2182-Common
- removed R901, R905, R909, R913: R_1, Resistor_SMD:R_0603_1608Metric, symbol Device:R_Small
- removed R902, R906, R910, R914: R_2, Resistor_SMD:R_0603_1608Metric, symbol Device:R_Small
- removed R903, R907, R911, R915: R_3, Resistor_SMD:R_0603_1608Metric, symbol Device:R_Small
- removed R904, R908, R912, R916: R_4, Resistor_SMD:R_0603_1608Metric, symbol Device:R_Small
- removed SW901: SW_A1, BVH_Switches:TacButton_6mm_6mm, symbol Switch:SW_Push_45deg
- removed SW902: SW_A2, BVH_Switches:TacButton_6mm_6mm, symbol Switch:SW_Push_45deg
- removed SW903: SW_A3, BVH_Switches:TacButton_6mm_6mm, symbol Switch:SW_Push_45deg
- removed SW904: SW_A4, BVH_Switches:TacButton_6mm_6mm, symbol Switch:SW_Push_45deg
- removed SW905: SW_B1, BVH_Switches:TacButton_6mm_6mm, symbol Switch:SW_Push_45deg
- removed SW906: SW_B2, BVH_Switches:TacButton_6mm_6mm, symbol Switch:SW_Push_45deg
- removed SW907: SW_B3, BVH_Switches:TacButton_6mm_6mm, symbol Switch:SW_Push_45deg
- removed SW908: SW_B4, BVH_Switches:TacButton_6mm_6mm, symbol Switch:SW_Push_45deg
- removed SW909: SW_C1, BVH_Switches:TacButton_6mm_6mm, symbol Switch:SW_Push_45deg
- removed SW910: SW_C2, BVH_Switches:TacButton_6mm_6mm, symbol Switch:SW_Push_45deg
- removed SW911: SW_C3, BVH_Switches:TacButton_6mm_6mm, symbol Switch:SW_Push_45deg
- removed SW912: SW_C4, BVH_Switches:TacButton_6mm_6mm, symbol Switch:SW_Push_45deg
- removed SW913: SW_D1, BVH_Switches:TacButton_6mm_6mm, symbol Switch:SW_Push_45deg
- removed SW914: SW_D2, BVH_Switches:TacButton_6mm_6mm, symbol Switch:SW_Push_45deg
- removed SW915: SW_D3, BVH_Switches:TacButton_6mm_6mm, symbol Switch:SW_Push_45deg
- removed SW916: SW_D4, BVH_Switches:TacButton_6mm_6mm, symbol Switch:SW_Push_45deg
- added S901: A1, BVH_Switches:TacButton_6mm_6mm_SK6812-E-Mini, symbol BVH_Switches_Inputs:Tac_Switch_With_Addressable_LED
- added S902: A2, BVH_Switches:TacButton_6mm_6mm_SK6812-E-Mini, symbol BVH_Switches_Inputs:Tac_Switch_With_Addressable_LED
- added S903: A3, BVH_Switches:TacButton_6mm_6mm_SK6812-E-Mini, symbol BVH_Switches_Inputs:Tac_Switch_With_Addressable_LED
- added S904: A4, BVH_Switches:TacButton_6mm_6mm_SK6812-E-Mini, symbol BVH_Switches_Inputs:Tac_Switch_With_Addressable_LED
- added S905: B1, BVH_Switches:TacButton_6mm_6mm_SK6812-E-Mini, symbol BVH_Switches_Inputs:Tac_Switch_With_Addressable_LED
- added S906: B2, BVH_Switches:TacButton_6mm_6mm_SK6812-E-Mini, symbol BVH_Switches_Inputs:Tac_Switch_With_Addressable_LED
- added S907: B3, BVH_Switches:TacButton_6mm_6mm_SK6812-E-Mini, symbol BVH_Switches_Inputs:Tac_Switch_With_Addressable_LED
- added S908: B4, BVH_Switches:TacButton_6mm_6mm_SK6812-E-Mini, symbol BVH_Switches_Inputs:Tac_Switch_With_Addressable_LED
- added S909: C1, BVH_Switches:TacButton_6mm_6mm_SK6812-E-Mini, symbol BVH_Switches_Inputs:Tac_Switch_With_Addressable_LED
- added S910: C2, BVH_Switches:TacButton_6mm_6mm_SK6812-E-Mini, symbol BVH_Switches_Inputs:Tac_Switch_With_Addressable_LED
- added S911: C3, BVH_Switches:TacButton_6mm_6mm_SK6812-E-Mini, symbol BVH_Switches_Inputs:Tac_Switch_With_Addressable_LED
- added S912: C4, BVH_Switches:TacButton_6mm_6mm_SK6812-E-Mini, symbol BVH_Switches_Inputs:Tac_Switch_With_Addressable_LED
- renumbered SW917 to S917
Connections:
- net +5V: now also S901.1 (VDD), S902.1 (VDD), S903.1 (VDD), S904.1 (VDD), S905.1 (VDD), S906.1 (VDD), S907.1 (VDD), S908.1 (VDD), S909.1 (VDD), S910.1 (VDD), S911.1 (VDD), S912.1 (VDD)
- net GND: now also S901.3 (GND), S901.6, S902.3 (GND), S902.6, S903.3 (GND), S903.6, S904.3 (GND), S904.6, S905.3 (GND), S905.6, S906.3 (GND), S906.6, S907.3 (GND), S907.6, S908.3 (GND), S908.6, S909.3 (GND), S909.6, S910.3 (GND), S910.6, S911.3 (GND), S911.6, S912.3 (GND), S912.6
- net RGB_DATA: now also S901.4 (DI)
- net ROW_A: now also S901.5, S902.5, S903.5, S904.5
- net ROW_B: now also S905.5, S906.5, S907.5, S908.5
- net ROW_C: now also S909.5, S910.5, S911.5, S912.5
- new net: S901.2 (DO), S902.4 (DI)
- new net: S905.2 (DO), S906.4 (DI)
- new net: S904.2 (DO), S905.4 (DI)
- new net: S911.2 (DO), S912.4 (DI)
- new net: S908.2 (DO), S909.4 (DI)
- new net: S907.2 (DO), S908.4 (DI)
- new net: S903.2 (DO), S904.4 (DI)
- new net: S909.2 (DO), S910.4 (DI)
- new net: S902.2 (DO), S903.4 (DI)
- new net: S910.2 (DO), S911.4 (DI)
- new net: S906.2 (DO), S907.4 (DI)
Other:
- moved on the sheet: S917
