File: hardware/prototype/minstro_combined_board/mpu_connectors.kicad_sch (KiCad schematic)
At the start: 6 parts, among them J401 FT6236_Conn_01x06, J402 ILI9488_Conn, J403 ST7789_Conn_01x12, Q401 2N7002

Commit message: Combined board started layout
Parts:
- renumbered J401 to J601, J402 to J602, J403 to J603, Q401 to Q601, R401 to R601, R402 to R602
Changed lines of the file:
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@@
 		(dnp no)
 		(fields_autoplaced yes)
-		(property "Reference" "#PWR0411"
+		(property "Reference" "#PWR0611"
 			(at 139.7 114.3 0)
 			(effects
@@
 			(project "display_board"
 				(path "/edc2d64f-9cdb-4ab0-b2de-c3cfa55e1c10/3cf64798-7e0b-4fcb-a543-023649f7a7ac"
-					(reference "#PWR0411")
+					(reference "#PWR0611")
 					(unit 1)
 				)
@@
 		(dnp no)
 		(fields_autoplaced yes)
-		(property "Reference" "#PWR0401"
+		(property "Reference" "#PWR0601"
 			(at 138.43 41.91 0)
 			(effects
@@
 			(project "display_board"
 				(path "/edc2d64f-9cdb-4ab0-b2de-c3cfa55e1c10/3cf64798-7e0b-4fcb-a543-023649f7a7ac"
-					(reference "#PWR0401")
+					(reference "#PWR0601")
 					(unit 1)
 				)
@@
 		(dnp no)
 		(fields_autoplaced yes)
-		(property "Reference" "#PWR0413"
+		(property "Reference" "#PWR0613"
 			(at 138.43 137.16 0)
 			(effects
@@
 			(project "display_board"
 				(path "/edc2d64f-9cdb-4ab0-b2de-c3cfa55e1c10/3cf64798-7e0b-4fcb-a543-023649f7a7ac"
-					(reference "#PWR0413")
+					(reference "#PWR0613")
 					(unit 1)
 				)
@@
 		(dnp no)
 		(fields_autoplaced yes)
-		(property "Reference" "#PWR0409"
+		(property "Reference" "#PWR0609"
 			(at 187.96 88.9 0)
 			(effects
@@
 			(project "display_board"
 				(path "/edc2d64f-9cdb-4ab0-b2de-c3cfa55e1c10/3cf64798-7e0b-4fcb-a543-023649f7a7ac"
-					(reference "#PWR0409")
+					(reference "#PWR0609")
 					(unit 1)
 				)
@@
 		(dnp no)
 		(fields_autoplaced yes)
-		(property "Reference" "#PWR0405"
+		(property "Reference" "#PWR0605"
 			(at 139.7 73.66 0)
 			(effects
@@
 			(project "display_board"
 				(path "/edc2d64f-9cdb-4ab0-b2de-c3cfa55e1c10/3cf64798-7e0b-4fcb-a543-023649f7a7ac"
-					(reference "#PWR0405")
+					(reference "#PWR0605")
 					(unit 1)
 				)
@@
 		(dnp no)
 		(fields_autoplaced yes)
-		(property "Reference" "#PWR0406"
+		(property "Reference" "#PWR0606"
 			(at 187.96 73.66 0)
 			(effects
@@
 			(project "display_board"
 				(path "/edc2d64f-9cdb-4ab0-b2de-c3cfa55e1c10/3cf64798-7e0b-4fcb-a543-023649f7a7ac"
-					(reference "#PWR0406")
+					(reference "#PWR0606")
 					(unit 1)
 				)
@@
 		(dnp no)
 		(fields_autoplaced yes)
-		(property "Reference" "#PWR0408"
+		(property "Reference" "#PWR0608"
 			(at 45.72 87.63 0)
 			(effects
@@
 			(project "display_board"
 				(path "/edc2d64f-9cdb-4ab0-b2de-c3cfa55e1c10/3cf64798-7e0b-4fcb-a543-023649f7a7ac"
-					(reference "#PWR0408")
+					(reference "#PWR0608")
 					(unit 1)
 				)
@@
 		(dnp no)
 		(fields_autoplaced yes)
-		(property "Reference" "#PWR0410"
+		(property "Reference" "#PWR0610"
 			(at 55.88 107.95 0)
 			(effects
@@
 			(project "display_board"
 				(path "/edc2d64f-9cdb-4ab0-b2de-c3cfa55e1c10/3cf64798-7e0b-4fcb-a543-023649f7a7ac"
-					(reference "#PWR0410")
+					(reference "#PWR0610")
 					(unit 1)
 				)
@@
 		(dnp no)
 		(fields_autoplaced yes)
-		(property "Reference" "#PWR0402"
+		(property "Reference" "#PWR0602"
 			(at 132.08 48.26 0)
 			(effects
@@
 			(project "display_board"
 				(path "/edc2d64f-9cdb-4ab0-b2de-c3cfa55e1c10/3cf64798-7e0b-4fcb-a543-023649f7a7ac"
-					(reference "#PWR0402")
+					(reference "#PWR0602")
 					(unit 1)
 				)
@@
 		(dnp no)
 		(fields_autoplaced yes)
-		(property "Reference" "J403"
+		(property "Reference" "J603"
 			(at 82.55 85.0899 0)
 			(effects
@@
 			(project ""
 				(path "/edc2d64f-9cdb-4ab0-b2de-c3cfa55e1c10/3cf64798-7e0b-4fcb-a543-023649f7a7ac"
-					(reference "J403")
+					(reference "J603")
 					(unit 1)
 				)
@@
 		(dnp no)
 		(fields_autoplaced yes)
-		(property "Reference" "#PWR0412"
+		(property "Reference" "#PWR0612"
 			(at 139.7 127 0)
 			(effects
@@
 			(project "display_board"
 				(path "/edc2d64f-9cdb-4ab0-b2de-c3cfa55e1c10/3cf64798-7e0b-4fcb-a543-023649f7a7ac"
-					(reference "#PWR0412")
+					(reference "#PWR0612")
 					(unit 1)
 				)
@@
 		(on_board yes)
 		(dnp no)
-		(property "Reference" "J402"
+		(property "Reference" "J602"
 			(at 167.386 78.74 90)
 			(effects
@@
 			(project ""
 				(path "/edc2d64f-9cdb-4ab0-b2de-c3cfa55e1c10/3cf64798-7e0b-4fcb-a543-023649f7a7ac"
-					(reference "J402")
+					(reference "J602")
 					(unit 1)
 				)
@@
 		(dnp no)
 		(fields_autoplaced yes)
-		(property "Reference" "R401"
+		(property "Reference" "R601"
 			(at 66.04 36.8299 0)
 			(effects
@@
 			(project ""
 				(path "/edc2d64f-9cdb-4ab0-b2de-c3cfa55e1c10/3cf64798-7e0b-4fcb-a543-023649f7a7ac"
-					(reference "R401")
+					(reference "R601")
 					(unit 1)
 				)
@@
 		(dnp no)
 		(fields_autoplaced yes)
-		(property "Reference" "J401"
+		(property "Reference" "J601"
 			(at 208.28 73.6599 0)
 			(effects
@@
 			(project ""
 				(path "/edc2d64f-9cdb-4ab0-b2de-c3cfa55e1c10/3cf64798-7e0b-4fcb-a543-023649f7a7ac"
-					(reference "J401")
+					(reference "J601")
 					(unit 1)
 				)
@@
 		(dnp no)
 		(fields_autoplaced yes)
-		(property "Reference" "#PWR0403"
+		(property "Reference" "#PWR0603"
 			(at 63.5 63.5 0)
 			(effects
@@
 			(project ""
 				(path "/edc2d64f-9cdb-4ab0-b2de-c3cfa55e1c10/3cf64798-7e0b-4fcb-a543-023649f7a7ac"
-					(reference "#PWR0403")
+					(reference "#PWR0603")
 					(unit 1)
 				)
@@
 		(dnp no)
 		(fields_autoplaced yes)
-		(property "Reference" "R402"
+		(property "Reference" "R602"
 			(at 50.8 44.45 90)
 			(effects
@@
 			(project "display_board"
 				(path "/edc2d64f-9cdb-4ab0-b2de-c3cfa55e1c10/3cf64798-7e0b-4fcb-a543-023649f7a7ac"
-					(reference "R402")
+					(reference "R602")
 					(unit 1)
 				)
@@
 		(dnp no)
 		(fields_autoplaced yes)
-		(property "Reference" "#PWR0407"
+		(property "Reference" "#PWR0607"
 			(at 45.72 82.55 0)
 			(effects
@@
 			(project ""
 				(path "/edc2d64f-9cdb-4ab0-b2de-c3cfa55e1c10/3cf64798-7e0b-4fcb-a543-023649f7a7ac"
-					(reference "#PWR0407")
+					(reference "#PWR0607")
 					(unit 1)
 				)
@@
 		(dnp no)
 		(fields_autoplaced yes)
-		(property "Reference" "#PWR0404"
+		(property "Reference" "#PWR0604"
 			(at 58.42 73.66 0)
 			(effects
@@
 			(project "display_board"
 				(path "/edc2d64f-9cdb-4ab0-b2de-c3cfa55e1c10/3cf64798-7e0b-4fcb-a543-023649f7a7ac"
-					(reference "#PWR0404")
+					(reference "#PWR0604")
 					(unit 1)
 				)
@@
 		(dnp no)
 		(fields_autoplaced yes)
-		(property "Reference" "Q401"
+		(property "Reference" "Q601"
 			(at 67.31 48.2599 0)
 			(effects
@@
 			(project ""
 				(path "/edc2d64f-9cdb-4ab0-b2de-c3cfa55e1c10/3cf64798-7e0b-4fcb-a543-023649f7a7ac"
-					(reference "Q401")
-					(unit 1)
-				)
+					(reference "Q601")
+					(unit 1)
+				)

Commit message: Schematic ERC complete
Connections:
- no-connect marks 1 -> 2
Changed lines of the file:
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@@
+	)
+	(no_connect
+		(at 148.59 57.15)
 	)
 	(no_connect

Commit message: Routing mostly completed
Parts:
- J601: value FT6236_Conn_01x06 -> FT6236
- J602: value ILI9488_Conn -> ILI9488
- J603: value ST7789_Conn_01x12 -> ST7789
Changed lines of the file:
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@@
 			)
 		)
-		(property "Value" "ST7789_Conn_01x12"
+		(property "Value" "ST7789"
 			(at 82.55 87.6299 0)
 			(effects
@@
 		)
 		(pin "11"
+		)
+		(pin "MP"
 		)
 		(instances
@@
 			)
 		)
-		(property "Value" "ILI9488_Conn"
+		(property "Value" "ILI9488"
 			(at 152.654 130.81 0)
 			(effects
@@
 		)
 		(pin "37"
+		)
+		(pin "MP"
 		)
 		(instances
@@
 			)
 		)
-		(property "Value" "FT6236_Conn_01x06"
+		(property "Value" "FT6236"
 			(at 208.28 76.1999 0)
 			(effects
@@
 		(pin "6"
 		)
+		(pin "MP"
+		)
 		(instances
