File: hardware/prototype/minstro_combined_board/hmi_nav_switch.kicad_sch (KiCad schematic)
At the start: 5 parts, among them J801 NAV CONN

Commit message: HMI processor firmware started
Parts:
- R801: value R_1 -> R_2
- R802: value R_2 -> R_4
- R803: value R_3 -> R_1
- R804: value R_4 -> R_3
Changed lines of the file:
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@@
 			)
 		)
-		(property "Value" "R_2"
+		(property "Value" "R_4"
 			(at 67.31 128.2699 0)
 			(effects
@@
 			)
 		)
-		(property "Value" "R_4"
+		(property "Value" "R_3"
 			(at 85.09 128.2699 0)
 			(effects
@@
 			)
 		)
-		(property "Value" "R_1"
+		(property "Value" "R_2"
 			(at 58.42 128.2699 0)
 			(effects
@@
 			)
 		)
-		(property "Value" "R_3"
+		(property "Value" "R_1"
 			(at 76.2 128.2699 0)
 			(effects
