File: hardware/prototype/minstro_combined_board/mpu_battery.kicad_sch (KiCad schematic)
At the start: 12 parts, among them J601 BATT, U601 BQ24074RGT

Commit message: Combined board started layout
Parts:
- renumbered C601 to C301, C602 to C302, C603 to C303, J601 to J301, R601 to R301, R602 to R302, R603 to R303, R604 to R304, R605 to R305, R606 to R306, R607 to R307, U601 to U301
Changed lines of the file:
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@@
 		(dnp no)
 		(fields_autoplaced yes)
-		(property "Reference" "R607"
+		(property "Reference" "R307"
 			(at 232.41 125.73 90)
 			(effects
@@
 			(project "display_board"
 				(path "/edc2d64f-9cdb-4ab0-b2de-c3cfa55e1c10/e86c5b72-a6ee-4f4b-b668-507d3abeaf42"
-					(reference "R607")
+					(reference "R307")
 					(unit 1)
 				)
@@
 		(dnp no)
 		(fields_autoplaced yes)
-		(property "Reference" "R604"
+		(property "Reference" "R304"
 			(at 111.76 92.71 90)
 			(effects
@@
 			(project "display_board"
 				(path "/edc2d64f-9cdb-4ab0-b2de-c3cfa55e1c10/e86c5b72-a6ee-4f4b-b668-507d3abeaf42"
-					(reference "R604")
+					(reference "R304")
 					(unit 1)
 				)
@@
 		(dnp no)
 		(fields_autoplaced yes)
-		(property "Reference" "C601"
+		(property "Reference" "C301"
 			(at 236.22 30.4863 0)
 			(effects
@@
 			(project "display_board"
 				(path "/edc2d64f-9cdb-4ab0-b2de-c3cfa55e1c10/e86c5b72-a6ee-4f4b-b668-507d3abeaf42"
-					(reference "C601")
+					(reference "C301")
 					(unit 1)
 				)
@@
 		(dnp no)
 		(fields_autoplaced yes)
-		(property "Reference" "#PWR0609"
+		(property "Reference" "#PWR0309"
 			(at 158.75 91.44 0)
 			(effects
@@
 			(project "display_board"
 				(path "/edc2d64f-9cdb-4ab0-b2de-c3cfa55e1c10/e86c5b72-a6ee-4f4b-b668-507d3abeaf42"
-					(reference "#PWR0609")
+					(reference "#PWR0309")
 					(unit 1)
 				)
@@
 		(dnp no)
 		(fields_autoplaced yes)
-		(property "Reference" "#PWR0614"
+		(property "Reference" "#PWR0314"
 			(at 111.76 148.59 0)
 			(effects
@@
 			(project "display_board"
 				(path "/edc2d64f-9cdb-4ab0-b2de-c3cfa55e1c10/e86c5b72-a6ee-4f4b-b668-507d3abeaf42"
-					(reference "#PWR0614")
+					(reference "#PWR0314")
 					(unit 1)
 				)
@@
 		(dnp no)
 		(fields_autoplaced yes)
-		(property "Reference" "R605"
+		(property "Reference" "R305"
 			(at 111.76 100.33 90)
 			(effects
@@
 			(project "display_board"
 				(path "/edc2d64f-9cdb-4ab0-b2de-c3cfa55e1c10/e86c5b72-a6ee-4f4b-b668-507d3abeaf42"
-					(reference "R605")
+					(reference "R305")
 					(unit 1)
 				)
@@
 		(dnp no)
 		(fields_autoplaced yes)
-		(property "Reference" "#PWR0615"
+		(property "Reference" "#PWR0315"
 			(at 111.76 154.94 0)
 			(effects
@@
 			(project "display_board"
 				(path "/edc2d64f-9cdb-4ab0-b2de-c3cfa55e1c10/e86c5b72-a6ee-4f4b-b668-507d3abeaf42"
-					(reference "#PWR0615")
+					(reference "#PWR0315")
 					(unit 1)
 				)
@@
 		(dnp no)
 		(fields_autoplaced yes)
-		(property "Reference" "R601"
+		(property "Reference" "R301"
 			(at 111.76 74.93 90)
 			(effects
@@
 			(project "display_board"
 				(path "/edc2d64f-9cdb-4ab0-b2de-c3cfa55e1c10/e86c5b72-a6ee-4f4b-b668-507d3abeaf42"
-					(reference "R601")
+					(reference "R301")
 					(unit 1)
 				)
@@
 		(dnp no)
 		(fields_autoplaced yes)
-		(property "Reference" "#PWR0605"
+		(property "Reference" "#PWR0305"
 			(at 257.81 41.91 0)
 			(effects
@@
 			(project "display_board"
 				(path "/edc2d64f-9cdb-4ab0-b2de-c3cfa55e1c10/e86c5b72-a6ee-4f4b-b668-507d3abeaf42"
-					(reference "#PWR0605")
+					(reference "#PWR0305")
 					(unit 1)
 				)
@@
 		(dnp no)
 		(fields_autoplaced yes)
-		(property "Reference" "#PWR0610"
+		(property "Reference" "#PWR0310"
 			(at 243.84 95.25 0)
 			(effects
@@
 			(project "display_board"
 				(path "/edc2d64f-9cdb-4ab0-b2de-c3cfa55e1c10/e86c5b72-a6ee-4f4b-b668-507d3abeaf42"
-					(reference "#PWR0610")
+					(reference "#PWR0310")
 					(unit 1)
 				)
@@
 		(dnp no)
 		(fields_autoplaced yes)
-		(property "Reference" "#PWR0608"
+		(property "Reference" "#PWR0308"
 			(at 158.75 83.82 0)
 			(effects
@@
 			(project "display_board"
 				(path "/edc2d64f-9cdb-4ab0-b2de-c3cfa55e1c10/e86c5b72-a6ee-4f4b-b668-507d3abeaf42"
-					(reference "#PWR0608")
+					(reference "#PWR0308")
 					(unit 1)
 				)
@@
 		(dnp no)
 		(fields_autoplaced yes)
-		(property "Reference" "#PWR0603"
+		(property "Reference" "#PWR0303"
 			(at 233.68 41.91 0)
 			(effects
@@
 			(project "display_board"
 				(path "/edc2d64f-9cdb-4ab0-b2de-c3cfa55e1c10/e86c5b72-a6ee-4f4b-b668-507d3abeaf42"
-					(reference "#PWR0603")
+					(reference "#PWR0303")
 					(unit 1)
 				)
@@
 		(dnp no)
 		(fields_autoplaced yes)
-		(property "Reference" "J601"
+		(property "Reference" "J301"
 			(at 254 63.4999 0)
 			(effects
@@
 			(project "display_board"
 				(path "/edc2d64f-9cdb-4ab0-b2de-c3cfa55e1c10/e86c5b72-a6ee-4f4b-b668-507d3abeaf42"
-					(reference "J601")
+					(reference "J301")
 					(unit 1)
 				)
@@
 		(dnp no)
 		(fields_autoplaced yes)
-		(property "Reference" "U601"
+		(property "Reference" "U301"
 			(at 140.5733 72.39 0)
 			(effects
@@
 			(project "display_board"
 				(path "/edc2d64f-9cdb-4ab0-b2de-c3cfa55e1c10/e86c5b72-a6ee-4f4b-b668-507d3abeaf42"
-					(reference "U601")
+					(reference "U301")
 					(unit 1)
 				)
@@
 		(dnp no)
 		(fields_autoplaced yes)
-		(property "Reference" "#PWR0602"
+		(property "Reference" "#PWR0302"
 			(at 257.81 31.75 0)
 			(effects
@@
 			(project "display_board"
 				(path "/edc2d64f-9cdb-4ab0-b2de-c3cfa55e1c10/e86c5b72-a6ee-4f4b-b668-507d3abeaf42"
-					(reference "#PWR0602")
+					(reference "#PWR0302")
 					(unit 1)
 				)
@@
 		(dnp no)
 		(fields_autoplaced yes)
-		(property "Reference" "#PWR0601"
+		(property "Reference" "#PWR0301"
 			(at 245.11 31.75 0)
 			(effects
@@
 			(project "display_board"
 				(path "/edc2d64f-9cdb-4ab0-b2de-c3cfa55e1c10/e86c5b72-a6ee-4f4b-b668-507d3abeaf42"
-					(reference "#PWR0601")
+					(reference "#PWR0301")
 					(unit 1)
 				)
@@
 		(dnp no)
 		(fields_autoplaced yes)
-		(property "Reference" "#PWR0611"
+		(property "Reference" "#PWR0311"
 			(at 102.87 114.3 0)
 			(effects
@@
 			(project "display_board"
 				(path "/edc2d64f-9cdb-4ab0-b2de-c3cfa55e1c10/e86c5b72-a6ee-4f4b-b668-507d3abeaf42"
-					(reference "#PWR0611")
+					(reference "#PWR0311")
 					(unit 1)
 				)
@@
 		(dnp no)
 		(fields_autoplaced yes)
-		(property "Reference" "R606"
+		(property "Reference" "R306"
 			(at 232.41 115.57 90)
 			(effects
@@
 			(project "display_board"
 				(path "/edc2d64f-9cdb-4ab0-b2de-c3cfa55e1c10/e86c5b72-a6ee-4f4b-b668-507d3abeaf42"
-					(reference "R606")
+					(reference "R306")
 					(unit 1)
 				)
@@
 		(dnp no)
 		(fields_autoplaced yes)
-		(property "Reference" "#PWR0604"
+		(property "Reference" "#PWR0304"
 			(at 245.11 41.91 0)
 			(effects
@@
 			(project "display_board"
 				(path "/edc2d64f-9cdb-4ab0-b2de-c3cfa55e1c10/e86c5b72-a6ee-4f4b-b668-507d3abeaf42"
-					(reference "#PWR0604")
+					(reference "#PWR0304")
 					(unit 1)
 				)
@@
 		(dnp no)
 		(fields_autoplaced yes)
-		(property "Reference" "C603"
+		(property "Reference" "C303"
 			(at 260.35 30.4863 0)
 			(effects
@@
 			(project "display_board"
 				(path "/edc2d64f-9cdb-4ab0-b2de-c3cfa55e1c10/e86c5b72-a6ee-4f4b-b668-507d3abeaf42"
-					(reference "C603")
+					(reference "C303")
 					(unit 1)
 				)
@@
 		(dnp no)
 		(fields_autoplaced yes)
-		(property "Reference" "#PWR0607"
+		(property "Reference" "#PWR0307"
 			(at 237.49 73.66 0)
 			(effects
@@
 			(project "display_board"
 				(path "/edc2d64f-9cdb-4ab0-b2de-c3cfa55e1c10/e86c5b72-a6ee-4f4b-b668-507d3abeaf42"
-					(reference "#PWR0607")
+					(reference "#PWR0307")
 					(unit 1)
 				)
@@
 		(dnp no)
 		(fields_autoplaced yes)
-		(property "Reference" "#PWR0606"
+		(property "Reference" "#PWR0306"
 			(at 224.79 68.58 0)
 			(effects
@@
 			(project "display_board"
 				(path "/edc2d64f-9cdb-4ab0-b2de-c3cfa55e1c10/e86c5b72-a6ee-4f4b-b668-507d3abeaf42"
-					(reference "#PWR0606")
+					(reference "#PWR0306")
 					(unit 1)
 				)
@@
 		(dnp no)
 		(fields_autoplaced yes)
-		(property "Reference" "#PWR0616"
+		(property "Reference" "#PWR0316"
 			(at 125.73 154.94 0)
 			(effects
@@
 			(project "display_board"
 				(path "/edc2d64f-9cdb-4ab0-b2de-c3cfa55e1c10/e86c5b72-a6ee-4f4b-b668-507d3abeaf42"
-					(reference "#PWR0616")
+					(reference "#PWR0316")
 					(unit 1)
 				)
@@
 		(dnp no)
 		(fields_autoplaced yes)
-		(property "Reference" "C602"
+		(property "Reference" "C302"
 			(at 247.65 30.4863 0)
 			(effects
@@
 			(project "display_board"
 				(path "/edc2d64f-9cdb-4ab0-b2de-c3cfa55e1c10/e86c5b72-a6ee-4f4b-b668-507d3abeaf42"
-					(reference "C602")
+					(reference "C302")
 					(unit 1)
 				)
@@
 		(dnp no)
 		(fields_autoplaced yes)
-		(property "Reference" "R603"
+		(property "Reference" "R303"
 			(at 111.76 82.55 90)
 			(effects
@@
 			(project "display_board"
 				(path "/edc2d64f-9cdb-4ab0-b2de-c3cfa55e1c10/e86c5b72-a6ee-4f4b-b668-507d3abeaf42"
-					(reference "R603")
+					(reference "R303")
 					(unit 1)
 				)
@@
 		(dnp no)
 		(fields_autoplaced yes)
-		(property "Reference" "#PWR0613"
+		(property "Reference" "#PWR0313"
 			(at 222.25 119.38 0)
 			(effects
@@
 			(project "display_board"
 				(path "/edc2d64f-9cdb-4ab0-b2de-c3cfa55e1c10/e86c5b72-a6ee-4f4b-b668-507d3abeaf42"
-					(reference "#PWR0613")
+					(reference "#PWR0313")
 					(unit 1)
 				)
@@
 		(dnp no)
 		(fields_autoplaced yes)
-		(property "Reference" "#PWR0612"
+		(property "Reference" "#PWR0312"
 			(at 138.43 115.57 0)
 			(effects
@@
 			(project "display_board"
 				(path "/edc2d64f-9cdb-4ab0-b2de-c3cfa55e1c10/e86c5b72-a6ee-4f4b-b668-507d3abeaf42"
-					(reference "#PWR0612")
+					(reference "#PWR0312")
 					(unit 1)
 				)
@@
 		(dnp no)
 		(fields_autoplaced yes)
-		(property "Reference" "R602"
+		(property "Reference" "R302"
 			(at 246.38 81.2799 0)
 			(effects
@@
 			(project "display_board"
 				(path "/edc2d64f-9cdb-4ab0-b2de-c3cfa55e1c10/e86c5b72-a6ee-4f4b-b668-507d3abeaf42"
-					(reference "R602")
-					(unit 1)
-				)
+					(reference "R302")
+					(unit 1)
+				)

Commit message: Layout and routing Power and initial signals, SD card
Parts:
- U301: footprint Package_DFN_QFN:VQFN-16-1EP_3x3mm_P0.5mm_EP1.6x1.6mm -> Package_DFN_QFN:VQFN-16-1EP_3x3mm_P0.5mm_EP1.6x1.6mm_ThermalVias
Connections:
- net BATT_TS: now also J301.1 (Pin_1); no longer J301.3 (Pin_3)
- net GND: now also J301.3 (Pin_3); no longer J301.1 (Pin_1)
Other:
- moved on the sheet: J301
Changed lines of the file:
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@@
 	(symbol
 		(lib_id "Connector:Conn_01x03_Pin")
-		(at 252.73 64.77 180)
+		(at 252.73 64.77 0)
+		(mirror y)
 		(unit 1)
 		(exclude_from_sim no)
@@
 		(on_board yes)
 		(dnp no)
-		(fields_autoplaced yes)
 		(property "Reference" "J301"
-			(at 254 63.4999 0)
+			(at 254 66.0401 0)
 			(effects
 				(font
@@
 		)
 		(property "Value" "BATT"
-			(at 254 66.0399 0)
+			(at 254 63.5001 0)
 			(effects
 				(font
@@
 			)
 		)
-		(property "Footprint" "Package_DFN_QFN:VQFN-16-1EP_3x3mm_P0.5mm_EP1.6x1.6mm"
+		(property "Footprint" "Package_DFN_QFN:VQFN-16-1EP_3x3mm_P0.5mm_EP1.6x1.6mm_ThermalVias"
 			(at 146.05 104.14 0)
 			(effects

Commit message: HMI processor firmware started
Parts:
- R301: value R_Small -> Rterm
- R304: value R_Small -> Rilm
- R305: value R_Small -> Riset
Other:
- note added: "Configuration Resistor Calculations: Riset = 0.25A = 3k5 Rilm = 0.1A = 15k5 - DNP when EN pins are 1,0 Rterm = 2k9 or DNP for default Rtmr = 6.5hr max charge time = 46k4"
Changed lines of the file:
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@@
 	(generator_version "9.0")
 	(paper "A4")
+	(text "Configuration Resistor Calculations:\n\nRiset = 0.25A = 3k5\nRilm = 0.1A = 15k5 - DNP when EN pins are 1,0\nRterm = 2k9 or DNP for default\nRtmr = 6.5hr max charge time = 46k4"
+		(exclude_from_sim no)
+		(at 138.176 124.968 0)
+		(effects
+			(font
+				(size 1.27 1.27)
+			)
+			(justify left)
+		)
+	)
 	(text "JST-PH 2.0\nRight Angle Connector"
 		(exclude_from_sim no)
@@
 			)
 		)
-		(property "Value" "R_Small"
+		(property "Value" "Rilm"
 			(at 111.76 95.25 90)
 			(effects
@@
 			)
 		)
-		(property "Value" "R_Small"
+		(property "Value" "Riset"
 			(at 111.76 102.87 90)
 			(effects
@@
 			)
 		)
-		(property "Value" "R_Small"
+		(property "Value" "Rterm"
 			(at 111.76 77.47 90)
 			(effects
